Commit message: Add frictionAnchor. Robots are now more stable than before.

File: tetrabot/urdf/tetrabot.urdf (robot description, URDF)
Before this commit: robot tetrabot, 17 links, 16 joints
Links:
- link base_link: mass 0.0265364970053473 -> 0.3005364970053473
- link leg1_joint1: mass 0.0141701030409731 -> 0.141701030409731
- link leg2_joint1: mass 0.0141701030409731 -> 0.141701030409731
- link leg3_joint1: mass 0.0141701030409731 -> 0.141701030409731
- link leg4_joint1: mass 0.0141701030409731 -> 0.141701030409731
